Commit message: modified boxer.xacro

File: boxer_description/urdf/boxer.xacro (robot description, xacro)
@@ -83,139 +83,169 @@
     <dynamics damping="100.0" friction="100"/>
   </joint>
+  <link name="top_mount_bottom">
+  	<visual>
+  		<origin xyz="0 0 0" rpy="0 0 0" />
+  		<geometry>
+  			<mesh filename="package://boxer_description/meshes/top_plate.stl" />
+  		</geometry>
+  		<material name="Boxer_DarkGrey" />
+  	</visual>
+  	<collision>
+  		<origin xyz="0 0 0" rpy="0 0 0" />
+  		<geometry>
+  			<mesh filename="package://boxer_description/meshes/top_plate_collision.stl" />
+  		</geometry>
+  	</collision>
+  </link>
+  <joint name="top_mount_bottom_joint" type="fixed">
+  	<origin xyz="0 0.1125 0" rpy="0 -1.5707 -1.5707" />
+  	<parent link="lift_link" />
+  	<child link="top_mount_bottom" />
+  </joint>
   <link name="top_mount">
-    <visual>
-      <origin xyz="0 0 0" rpy="0 0 0" />
-      <geometry>
-        <mesh filename="package://boxer_description/meshes/top_plate.stl" />
-      </geometry>
-      <material name="Boxer_DarkGrey" />
-    </visual>
-    <collision>
-      <origin xyz="0 0 0" rpy="0 0 0" />
-      <geometry>
-        <mesh filename="package://boxer_description/meshes/top_plate_collision.stl" />
-      </geometry>
-    </collision>
-  </link>
+  	<visual>
+  		<origin xyz="0 0 0" rpy="0 0 0" />
+  		<geometry>
+  			<mesh filename="package://boxer_description/meshes/top_plate.stl" />
+  		</geometry>
+  		<material name="Boxer_DarkGrey" />
+  	</visual>
+  	<collision>
+  		<origin xyz="0 0 0" rpy="0 0 0" />
+  		<geometry>
+  			<mesh filename="package://boxer_description/meshes/top_plate_collision.stl" />
+  		</geometry>
+  	</collision>
+  </link>
+  <!-- 0.27 in z direction because extrusion is 0.30, and plate is 0.1 -->
   <joint name="top_mount_joint" type="fixed">
-    <origin xyz="0 0.1125 0" rpy="0 -1.5707 -1.5707" />
-    <parent link="lift_link" />
-    <child link="top_mount" />
+  	<origin xyz="0.2785 -0.1835 0.31" rpy="0 0 0" />
+  	<parent link="extrusion1" />
+  	<child link="top_mount" />
   </joint>
   <link name="rotacastor_right_link">
-    <inertial>
-      <origin xyz="0 0 0" rpy="0 0 0"/>
-      <mass value="100"/>
-      <inertia ixx="0.2" ixy="0" ixz="0" iyy="0.2" iyz="0" izz="0.2"/>
-    </inertial>
-    <visual>
-      <origin xyz="0 0 0" rpy="0 1.5708 0" />
-      <geometry>
-        <cylinder radius="0.0625" length="0.06" />
-      </geometry>
-      <material name="Boxer_Red"/>
-    </visual>
-    <collision>
-      <origin xyz="0 0 0" rpy="0 1.5708 0" />
-      <geometry>
-        <cylinder radius="0.0625" length="0.001" />
-      </geometry>
-    </collision>
+  	<inertial>
+  		<origin xyz="0 0 0" rpy="0 0 0"/>
+  		<mass value="100"/>
+  		<inertia ixx="0.2" ixy="0" ixz="0" iyy="0.2" iyz="0" izz="0.2"/>
+  	</inertial>
+  	<visual>
+  		<origin xyz="0 0 0" rpy="0 1.5708 0" />
+  		<geometry>
+  			<cylinder radius="0.0625" length="0.06" />
+  		</geometry>
+  		<material name="Boxer_Red"/>
+  	</visual>
+  	<collision>
+  		<origin xyz="0 0 0" rpy="0 1.5708 0" />
+  		<geometry>
+  			<cylinder radius="0.0625" length="0.001" />
+  		</geometry>
+  	</collision>
   </link>
   <joint name="rotacastor_right_joint" type="fixed">
-    <origin xyz="-0.177 -0.274 0.043" rpy="0 0 0" />
-    <parent link="chassis_link" />
-    <child link="rotacastor_right_link" />
-    <axis  xyz="1 0 0" />
-    <dynamics damping="1.0" />
+  	<origin xyz="-0.177 -0.274 0.043" rpy="0 0 0" />
+  	<parent link="chassis_link" />
+  	<child link="rotacastor_right_link" />
+  	<axis  xyz="1 0 0" />
+  	<dynamics damping="1.0" />
   </joint>
   <link name="rotacastor_left_link">
-    <inertial>
-      <origin xyz="0 0 0" rpy="0 0 0"/>
-      <mass value="100"/>
-      <inertia ixx="0.2" ixy="0" ixz="0" iyy="0.2" iyz="0" izz="0.2"/>
-    </inertial>
-    <visual>
-      <origin xyz="0 0 0" rpy="0 1.5708 0" />
-      <geometry>
-        <cylinder radius="0.0625" length="0.06" />
-      </geometry>
-      <material name="Boxer_Red"/>
-    </visual>
-    <collision>
-      <origin xyz="0 0 0" rpy="0 1.5708 0" />
-      <geometry>
-        <cylinder radius="0.0625" length="0.001" />
-      </geometry>
-    </collision>
+  	<inertial>
+  		<origin xyz="0 0 0" rpy="0 0 0"/>
+  		<mass value="100"/>
+  		<inertia ixx="0.2" ixy="0" ixz="0" iyy="0.2" iyz="0" izz="0.2"/>
+  	</inertial>
+  	<visual>
+  		<origin xyz="0 0 0" rpy="0 1.5708 0" />
+  		<geometry>
+  			<cylinder radius="0.0625" length="0.06" />
+  		</geometry>
+  		<material name="Boxer_Red"/>
+  	</visual>
+  	<collision>
+  		<origin xyz="0 0 0" rpy="0 1.5708 0" />
+  		<geometry>
+  			<cylinder radius="0.0625" length="0.001" />
+  		</geometry>
+  	</collision>
   </link>
   <joint name="rotacastor_left_joint" type="fixed">
-    <origin xyz="0.177 -0.274 0.043" rpy="0 0 0" />
-    <parent link="chassis_link" />
-    <child link="rotacastor_left_link" />
-    <axis xyz="1 0 0" />
-    <dynamics damping="1.0" />
+  	<origin xyz="0.177 -0.274 0.043" rpy="0 0 0" />
+  	<parent link="chassis_link" />
+  	<child link="rotacastor_left_link" />
+  	<axis xyz="1 0 0" />
+  	<dynamics damping="1.0" />
   </joint>
   <link name="wheel_right_link">
-    <inertial>
-      <origin xyz="0 0 0" rpy="0 0 0"/>
-      <mass value="100"/>
-      <inertia ixx="0.2" ixy="0" ixz="0" iyy="0.2" iyz="0" izz="0.2"/>
-    </inertial>
-    <visual>
-      <origin xyz="0 0 0" rpy="0 1.5708 0" />
-      <geometry>
-        <cylinder radius="0.080" length="0.05" />
-      </geometry>
-      <material name="Boxer_Red"/>
-    </visual>
-    <collision>
-      <origin xyz="0 0 0" rpy="0 1.5708 0" />
-      <geometry>
-        <cylinder radius="0.080" length="0.001" />
-      </geometry>
-    </collision>
+  	<inertial>
+  		<origin xyz="0 0 0" rpy="0 0 0"/>
+  		<mass value="100"/>
+  		<inertia ixx="0.2" ixy="0" ixz="0" iyy="0.2" iyz="0" izz="0.2"/>
+  	</inertial>
+  	<visual>
+  		<origin xyz="0 0 0" rpy="0 1.5708 0" />
+  		<geometry>
+  			<cylinder radius="0.080" length="0.05" />
+  		</geometry>
+  		<material name="Boxer_Red"/>
+  	</visual>
+  	<collision>
+  		<origin xyz="0 0 0" rpy="0 1.5708 0" />
+  		<geometry>
+  			<cylinder radius="0.080" length="0.001" />
+  		</geometry>
+  	</collision>
   </link>
   <joint name="wheel_right_joint" type="continuous">
-    <origin xyz="-0.247 0.157 0.058" rpy="0 0 0" />
-    <parent link="chassis_link" />
-    <child link="wheel_right_link" />
-    <axis xyz="1 0 0" />
-    <dynamics damping="1.0" />
+  	<origin xyz="-0.247 0.157 0.058" rpy="0 0 0" />
+  	<parent link="chassis_link" />
+  	<child link="wheel_right_link" />
+  	<axis xyz="1 0 0" />
+  	<limit effort="10000" velocity="1000"/>
+  	<dynamics damping="1.0" />
   </joint>
   <link name="wheel_left_link">
-    <inertial>
-      <origin xyz="0 0 0" rpy="0 0 0"/>
-      <mass value="100"/>
-      <inertia ixx="0.2" ixy="0" ixz="0" iyy="0.2" iyz="0" izz="0.2"/>
-    </inertial>
-    <visual>
-      <origin xyz="0 0 0" rpy="0 1.5708 0" />
-      <geometry>
-        <cylinder radius="0.080" length="0.05" />
-      </geometry>
-      <material name="Boxer_Red"/>
-    </visual>
-    <collision>
-      <origin xyz="0 0 0" rpy="0 1.5708 0" />
-      <geometry>
-        <cylinder radius="0.080" length="0.001" />
-      </geometry>
-    </collision>
+  	<inertial>
+  		<origin xyz="0 0 0" rpy="0 0 0"/>
+  		<mass value="100"/>
+  		<inertia ixx="0.2" ixy="0" ixz="0" iyy="0.2" iyz="0" izz="0.2"/>
+  	</inertial>
+  	<visual>
+  		<origin xyz="0 0 0" rpy="0 1.5708 0" />
+  		<geometry>
+  			<cylinder radius="0.080" length="0.05" />
+  		</geometry>
+  		<material name="Boxer_Red"/>
+  	</visual>
+  	<collision>
+  		<origin xyz="0 0 0" rpy="0 1.5708 0" />
+  		<geometry>
+  			<cylinder radius="0.080" length="0.001" />
+  		</geometry>
+  	</collision>
   </link>
   <joint name="wheel_left_joint" type="continuous">
-    <origin xyz="0.247 0.157 0.058" rpy="0 0 0" />
-    <parent link="chassis_link" />
-    <child link="wheel_left_link" />
-    <axis xyz="1 0 0" />
-    <dynamics damping="1.0" />
+  	<origin xyz="0.247 0.157 0.058" rpy="0 0 0" />
+  	<parent link="chassis_link" />
+  	<child link="wheel_left_link" />
+  	<axis xyz="1 0 0" />
+  	<limit effort="10000" velocity="1000"/>
+  	<dynamics damping="1.0" />
   </joint>
   <!-- Base link with no geometry or inertia, because KDL needs it
-      to be that way. -->
+  to be that way. -->
   <link name="base_link" />
   <joint name="base_chassis_joint" type="fixed">
-    <origin xyz="0.15 0 0" rpy="0 0 1.5708" />
+  	<origin xyz="0.15 0 0" rpy="0 0 1.5708" />
+  	<parent link="base_link" />
+  	<child link="chassis_link" />
+  </joint>
+  <!-- link for collision avoidance-->
+  <link name="base_sphere" />
+  <joint name="base_sphere_joint=" type="fixed">
+    <origin xyz="0.15 0 0.25" />
     <parent link="base_link" />
-    <child link="chassis_link" />
+    <child link="base_sphere" />
   </joint>
   <!-- Projection of base_link on the ground to get the 3D data
@@ -223,82 +253,93 @@
   <link name="base_footprint" />
   <joint name="base_footprint_joint" type="fixed">
-    <origin xyz="0 0 -0.08" rpy="0 0 0" />
-    <parent link="base_link" />
-    <child link="base_footprint" />
+  	<origin xyz="0 0 -0.08" rpy="0 0 0" />
+  	<parent link="base_link" />
+  	<child link="base_footprint" />
   </joint>
   <!-- Link for the position of the laser. -->
   <link name="front_laser" />
   <joint name="base_laser_joint" type="fixed">
-    <!-- LIDAR is moved forward slightly, from 0.407, to mitigate collision with internal_link due to slow physics updates  -->
-    <origin xyz="0.44 0 0.172" rpy="3.14159 0 0" />
-    <parent link="base_link" />
-    <child link="front_laser" />
+  	<!-- LIDAR is moved forward slightly, from 0.407, to mitigate collision with internal_link due to slow physics updates  -->
+  	<origin xyz="0.44 0 0.172" rpy="3.14159 0 0" />
+  	<parent link="base_link" />
+  	<child link="front_laser" />
   </joint>
   <!-- Stereo camera link to base_link. -->
   <link name="stereo" />
   <joint name="stereo_camera_joint" type="fixed">
-    <origin xyz="0.4884 0 0.05465" rpy="3.14159 0 0" />
-    <parent link="base_link" />
-    <child link="stereo" />
+  	<origin xyz="0.4884 0 0.05465" rpy="3.14159 0 0" />
+  	<parent link="base_link" />
+  	<child link="stereo" />
   </joint>
   <link name="stereo_left" />
   <joint name="stereo_left_joint" type="fixed">
-    <origin xyz="0 0.060 0" rpy="-1.570796327 0 -1.570796327" />
-    <parent link="stereo" />
-    <child link="stereo_left" />
+  	<origin xyz="0 0.060 0" rpy="-1.570796327 0 -1.570796327" />
+  	<parent link="stereo" />
+  	<child link="stereo_left" />
   </joint>
   <link name="stereo_right" />
   <joint name="stereo_right_joint" type="fixed">
-    <origin xyz="0 -0.060 0" rpy="-1.570796327 0 -1.570796327" />
-    <parent link="stereo" />
-    <child link="stereo_right" />
+  	<origin xyz="0 -0.060 0" rpy="-1.570796327 0 -1.570796327" />
+  	<parent link="stereo" />
+  	<child link="stereo_right" />
+  </joint>
+  <link name="top_camera" />
+  <joint name="top_camera_joint" type="fixed">
+  	<origin xyz="0.1 0 0.3" rpy="0 ${-0/10} 0" />
+  	<parent link="top_mount" />
+  	<child link="top_camera" />
+  </joint>
+  <link name="depth_camera" />
+  <joint name="depth_camera_joint" type="fixed">
+  	<origin xyz="0.1 0 0.1" rpy="${-pi/2} 0 ${-pi/2}" />
+  	<parent link="top_camera" />
+  	<child link="depth_camera" />
   </joint>
   <!-- Sonar links to base link joints -->
   <link name="rear_left_sonar_link" />
   <joint name="rear_left_sonar_joint" type="fixed">
-    <origin xyz="-0.2043 0.150 0.157" rpy="0 0 3.14159" />
-    <parent link="base_link" />
-    <child link="rear_left_sonar_link" />
+  	<origin xyz="-0.2043 0.150 0.157" rpy="0 0 3.14159" />
+  	<parent link="base_link" />
+  	<child link="rear_left_sonar_link" />
   </joint>
   <link name="rear_right_sonar_link" />
   <joint name="rear_right_sonar_joint" type="fixed">
-    <origin xyz="-0.2043 -0.150 0.157" rpy="0 0 3.141597" />
-    <parent link="base_link" />
-    <child link="rear_right_sonar_link" />
+  	<origin xyz="-0.2043 -0.150 0.157" rpy="0 0 3.141597" />
+  	<parent link="base_link" />
+  	<child link="rear_right_sonar_link" />
   </joint>
   <transmission name="wheel_left_transmission">
-    <type>transmission_interface/SimpleTransmission</type>
-    <joint name="wheel_left_joint">
-      <hardwareInterface>hardware_interface/VelocityJointInterface</hardwareInterface>
-    </joint>
-    <actuator name="wheel_left_actuator">
-      <mechanicalReduction>1</mechanicalReduction>
-    </actuator>
+  	<type>transmission_interface/SimpleTransmission</type>
+  	<joint name="wheel_left_joint">
+  		<hardwareInterface>hardware_interface/VelocityJointInterface</hardwareInterface>
+  	</joint>
+  	<actuator name="wheel_left_actuator">
+  		<mechanicalReduction>1</mechanicalReduction>
+  	</actuator>
   </transmission>
   <transmission name="wheel_right_transmission">
-    <type>transmission_interface/SimpleTransmission</type>
-    <joint name="wheel_right_joint">
-      <hardwareInterface>hardware_interface/VelocityJointInterface</hardwareInterface>
-    </joint>
-    <actuator name="wheel_right_actuator">
-      <mechanicalReduction>1</mechanicalReduction>
-    </actuator>
+  	<type>transmission_interface/SimpleTransmission</type>
+  	<joint name="wheel_right_joint">
+  		<hardwareInterface>hardware_interface/VelocityJointInterface</hardwareInterface>
+  	</joint>
+  	<actuator name="wheel_right_actuator">
+  		<mechanicalReduction>1</mechanicalReduction>
+  	</actuator>
   </transmission>
   <transmission name="lift_transmission">
-    <type>transmission_interface/SimpleTransmission</type>
-    <joint name="lift_joint">
-      <hardwareInterface>hardware_interface/PositionJointInterface</hardwareInterface>
-    </joint>
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